File: mixer.kicad_sch (KiCad schematic)
At the start: 16 parts, among them U2 CD74HC4052E, U3 MCP6002-xP

Commit message: Update kicad to rev 0.1
Connections:
- net OSC-IN-1 renamed OSC-1-IN
- net OSC-IN-2 renamed OSC-2-IN
Other:
- note added: "Signalförstärkning"
- note added: "Tayloe-mixer"
- moved on the sheet: C10, C11, C12, C13, C5, C7, R10, R11, R12, R13, R14, R15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
