File: power-supply.kicad_sch (KiCad schematic)
At the start: 12 parts, among them J1 Barrel_Jack, Q1 IRF9540N, U1 L7805

Commit message: Update kicad to rev 0.1
Other:
- note added: "Skyddsdiod"
Changed lines of the file:
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@@
+		)
+	)
+	(text "Skyddsdiod"
+		(exclude_from_sim no)
+		(at 151.13 72.39 0)
+		(effects
+			(font
+				(size 1.27 1.27)
+			)
 		)
 	)
