File: projekt-am.kicad_sch (KiCad schematic)
At the start: 0 parts

Commit message: Update kicad to rev 0.1
Other:
- sheet LC Tank Circuit ports: added PWM_TUNING_INPUT; removed PWM_TUNING
- sheet MCU ports: added I_SIGNAL_INPUT, OSC-1-OUT, OSC-2-OUT, PWM_AUDIO_OUTPUT, PWM_TUNING_OUTPUT, Q_SIGNAL_INPUT; removed none
- sheet Mixer ports: added OSC-1-IN, OSC-2-IN; removed OSC-IN-1, OSC-IN-2
