File: mcu.kicad_sch (KiCad schematic)
At the start: 0 parts

Commit message: Update kicad to rev 0.1
Parts:
- added C18, C19, C20, C24: 100 nF, symbol Device:C_Small
- added C21, C22: 22 pF, symbol Device:C_Small
- added C23, C25: 10nF, symbol Device:C_Small
- added C26: 10 nF, symbol Device:C_Small
- added J3: AVR-ISP-6, symbol Connector:AVR-ISP-6
- added R20, R21, R22, R23: 10k, symbol Device:R
- added SW1: SW_Omron_B3FS, symbol Switch:SW_Omron_B3FS
- added SW2: RotaryEncoder_Switch, symbol Device:RotaryEncoder_Switch
- added U5: ATmega328P-P, Package_DIP:DIP-28_W7.62mm, symbol MCU_Microchip_ATmega:ATmega328P-P
- added Y1: Si5351A-B-GT, Package_SO:MSOP-10_3x3mm_P0.5mm, symbol Oscillator:Si5351A-B-GT
- added Y2: 16 MHz, symbol Device:Crystal
Connections:
- new net: C22.1, U5.10 (XTAL2/PB7), Y2.1
- new net: C18.1, U5.21 (AREF)
- new net: C21.1, U5.9 (XTAL1/PB6), Y2.2
- new net +5V: C19.2, C20.2, C24.1, J3.2 (VCC), R20.1, R21.1, R22.1, R23.1, U5.20 (AVCC), U5.7 (VCC), Y1.1 (VDD)
- new net GND: C18.2, C19.1, C20.1, C21.2, C22.2, C23.2, C24.2, C25.2, C26.2, J3.6 (GND), SW1.2, SW2.C, SW2.S2, U5.22 (GND), U5.8 (GND), Y1.8 (GND)
- new net ISP_MISO: J3.1 (MISO), U5.18 (PB4)
- new net ISP_MOSI: J3.4 (MOSI), U5.17 (PB3)
- new net ISP_RESET: J3.5 (~{RST}), R20.2, SW1.1, U5.1 (~{RESET}/PC6)
- new net ISP_SCK: J3.3 (SCK), U5.19 (PB5)
- new net I_SIGNAL_INPUT: U5.23 (PC0)
- new net OSC-1-OUT: Y1.10 (CLK0)
- new net OSC-2-OUT: Y1.9 (CLK1)
- new net PC4/SDA: U5.27 (PC4), Y1.5 (SDA)
- new net PC5/SCL: U5.28 (PC5), Y1.4 (SCL)
- new net PWM_AUDIO_OUTPUT: U5.5 (PD3)
- new net PWM_TUNING_OUTPUT: U5.16 (PB2)
- new net Q_SIGNAL_INPUT: U5.24 (PC1)
- new net ROTARY_A: C26.1, R21.2, SW2.A, U5.4 (PD2)
- new net ROTARY_B: C25.1, R23.2, SW2.B, U5.13 (PD7)
- new net ROTARY_SWITCH: C23.1, R22.2, SW2.S1, U5.11 (PD5)
- no-connect marks 0 -> 12
Other:
- note added: "Dithering?"
- note added: "ISP Header (För ATMEL-ICE)"
- note added: "MCU (ATMega328p)"
- note added: "PD2 (INT0 - interrupt 0)"
- note added: "Reset-switch"
- note added: "Rotary encoder (Används för att kontrollera tuning)"
- note added: "SI5351A breakout (Lokal Oscillator)"
